File: swag-badge(Backup).kicad_pcb (KiCad board)
At the start: 2 copper layers, 80 x 120 mm, 28 parts, among them J1 OLED_1, J10 IO15 T3, J11 IO12 T5, J12 Breakout_LHS, J13 Breakout_RHS, J2 OLED_2, J3 SAO_2, J4 SAO_1, J5 SAO_4, J6 SAO_3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

Commit message: SAOs rotated 45° Silks updated
Credits still need to be verified
Parts:
- removed G***: LOGO, SwagBadge:Logo_LCA2021_05_Smaller
- added L1: Logo_LCA2021, SwagBadge:Logo_LCA2021_04A, F.Cu at (40.0, -64.0)
- moved J5 10.0 mm to (74.0, -80.0), turned to 270 degrees
- moved J6 10.0 mm to (6.00, -80.0), turned to 90 degrees
Routing:
- net /GPIO4: track 254.8 -> 230.4 mm
- net /GPIO25: track 115.2 -> 102.2 mm
- net /GPIO5: track 260.1 -> 247.5 mm
- net /GPIO23: track 100.0 -> 91.6 mm
- net /GPIO26: track 110.1 -> 104.4 mm
- net /GPIO18: track 103.8 -> 105.1 mm
Other:
- board text added: "@swagbadge"
- board text removed: "@swagbadge2021"
- board text removed: "CHARGE"
- board text removed: "LED"
